Commit message: correcct obj file path in this file

File: urdf/dart.urdf (robot description, URDF)
Before this commit: robot UR_grasp_sim, 1 links, 0 joints
Links:
- link base: geometry collision mesh filename=./urdf/ProDart_JB_vhacd.obj scale=1 1 1; visual mesh filename=./urdf/ProDart_JB.obj scale=1 1 1
