Commit message: correcct obj file path in this file

File: urdf/dartboard.urdf (robot description, URDF)
Before this commit: robot UR_grasp_sim, 1 links, 0 joints
Links:
- link _name: geometry collision mesh filename=./urdf/dart_tarcza_obj_vhacd.obj scale=0.05 0.05 0.05; visual mesh filename=./urdf/dart_tarcza_obj.obj scale=0.05 0.05 0.05

Commit message: train_RL

File: urdf/dartboard.urdf (robot description, URDF)
Before this commit: robot UR_grasp_sim, 1 links, 0 joints
Links:
- removed link _name
- added link dartboard, mass 1.0; collision mesh filename=./urdf/dart_tarcza_obj_vhacd.obj scale=0.05 0.05 0.05; visual mesh filename=./urdf/dart_tarcza_obj.obj scale=0.05 0.05 0.05
